File: pcb/node-pcb/node-pcb.kicad_pcb (KiCad board)
At the start: 4 copper layers, 44 x 44 mm, 55 parts, among them J1 TYPE-C-31-M-12, J2 BM08B-GHS-TBT(LF)(SN), J3 BM08B-GHS-TBT(LF)(SN), J4 TC2030, J5 AFC11-S12ICA-00, Q1 S8050, SW1 TS-1187A-B-A-B, U1 AP2112K-3.3, U2 W25Q32JVSSIQ, U3 RP2040, U4 THVD1450DR, Y1 ABM8-272-T3

Commit message: - Updated PCB design - added link to CAD files
Parts:
- moved C16 7.52 mm to (110.5, 111.5), turned to -90 degrees
- moved C11 6.96 mm to (106.5, 112.5), turned to 0 degrees
- moved TP1 6.40 mm to (111.5, 85.5)
- moved R16 3.50 mm to (112.0, 107.5)
- moved R17 3.00 mm to (112.0, 106.0)
- moved R5 2.00 mm to (90.0, 84.0)
- moved SW1 1.58 mm to (84.0, 86.0)
- moved C10 1.50 mm to (100.0, 119.0), turned to 0 degrees
- moved D1 1.50 mm to (107.0, 115.0)
- moved R6 1.12 mm to (84.5, 91.0), turned to 0 degrees
- moved C19 0.50 mm to (93.5, 116.5)
Routing:
- net 5V_LOCAL: track 51.8 -> 41.0 mm
- net /ADDR_IN: track 27.4 -> 23.3 mm
- net /SPARE_IN: track 23.2 -> 20.1 mm
- net +3V3: track 63.4 -> 60.5 mm
- net +5V_BUS: track 22.8 -> 25.5 mm
- net /QSPI_SS: track 30.7 -> 28.4 mm
- net Net-(J3-Pad2): track 2.92 -> 4.89 mm
- net Net-(J3-Pad1): track 3.13 -> 4.82 mm
- net GND: track 104.9 -> 106.3 mm
Other:
- outline, holes or cut-outs redrawn
